Commit message: - Refactoring the urdf dscription recorrding to hydrus package - Add upboard based model

File: robots/dragon/robots/quad/upboard_sensors_201911/robot.gazebo.xacro (robot description, xacro)
@@ -3,7 +3,6 @@
     xmlns:xacro="http://www.ros.org/wiki/xacro" name="dragon" >
   <!-- robot urdf -->
-  <xacro:include filename="$(find dragon)/robots/quad/euclid_201709.urdf.xacro" />
+  <xacro:include filename="$(find dragon)/robots/quad/upboard_sensors_201911/robot.urdf.xacro" />
   <!-- gazebo plugin for sensors -->
-  <!-- temporary -->
   <xacro:include filename="$(find dragon)/robots/default.gazebo.xacro" />
 </robot>

File: robots/dragon/urdf/dragon_common.xacro (robot description, xacro)
@@ -14,4 +14,22 @@
   <!-- dynamics -->
   <xacro:property name="max_force" value="30" /> <!-- [N] -->
+  <xacro:macro name="extra_module" params="name parent *origin *inertial visible:=0 model_url:=1 scale:=1">
+    <joint name="${parent}2${name}" type="fixed">
+      <parent link="${parent}"/>
+      <child link="${name}"/>
+      <xacro:insert_block name="origin" />
+    </joint>
+    <link name="${name}">
+      <xacro:insert_block name="inertial" />
+      <xacro:if value="${visible == 1}">
+        <visual>
+          <origin rpy="0 0 0" xyz="0 0 0"/>
+          <geometry>
+            <mesh filename="${model_url}" scale= "${scale} ${scale} ${scale}"/>
+          </geometry>
+        </visual>
+      </xacro:if>
+    </link>
+  </xacro:macro>
   <xacro:macro name="link_model" params="type">
     <!-- box collision geometry does not work well for FCL -->

File: robots/dragon/urdf/dragon_link.urdf.xacro (robot description, xacro)
@@ -9,13 +9,9 @@
       <xacro:if value="${self == 1}">
         <inertial>
-          <origin xyz="${link_length* 0.5 + 20.63 * 0.001} ${-7.10 * 0.001} ${-24.66 * 0.001}" rpy="0 0 0"/>
-          <mass value="0.7485" />
-          <!-- bad problem: https://github.com/tongtybj/aerial_robot/issues/155
+          <origin xyz="${link_length* 0.5 + 0.020630} -0.007100 -0.024660" rpy="0 0 0"/>
+          <mass value="0.748500"/>
           <inertia
-              ixx="0.0014" iyy="0.0154" izz="0.0147"
-              ixy="-0.0008" ixz="0.0006" iyz="0.0"/> -->
-          <inertia
-              ixx="0.0009" iyy="0.0146" izz="0.0143"
-              ixy="-0.0009" ixz="0.0002" iyz="0.0001"/>
+              ixx="0.000907" iyy="0.014523" izz="0.014238"
+              ixy="-0.001008" ixz="0.000152" iyz="0.000131"/>
         </inertial>
         <xacro:link_model type="head_link" />
@@ -25,13 +21,9 @@
         <xacro:if value="${self == child}">
           <inertial>
-            <origin xyz="${link_length* 0.5 - 47.26 * 0.001} ${-0.12 * 0.001} ${-17.74 * 0.001}" rpy="0 0 0"/>
-            <mass value="0.7460" />
-            <!-- bad problem: https://github.com/tongtybj/aerial_robot/issues/155
+            <origin xyz="${link_length* 0.5 -0.047260} -0.000120 -0.017740" rpy="0 0 0"/>
+            <mass value="0.746000"/>
             <inertia
-                ixx="0.0014" iyy="0.0158" izz="0.0145"
-                ixy="0.0" ixz="-0.0006" iyz="0.0"/> -->
-            <inertia
-                ixx="0.0012" iyy="0.0139" izz="0.0128"
-                ixy="0.0" ixz="0.0" iyz="0.0"/>
+                ixx="0.001165" iyy="0.013875" izz="0.012844"
+                ixy="0.000002" ixz="0.000068" iyz="0.000002"/>
           </inertial>
           <xacro:link_model type="end_link" />
@@ -41,13 +33,9 @@
           <xacro:if value="${baselink}">
             <inertial>
-              <origin xyz="${link_length* 0.5 + 11.73 * 0.001} ${-4.91 * 0.001} ${-13.87 * 0.001}" rpy="0 0 0"/>
-              <mass value="1.096" />
-              <!-- bad problem: https://github.com/tongtybj/aerial_robot/issues/155
+              <origin xyz="${link_length* 0.5 -0.014560} -0.006040 -0.014650" rpy="0 0 0"/>
+              <mass value="0.890000"/>
               <inertia
-                  ixx="0.0019" iyy="0.0226" izz="0.0217"
-                  ixy="-0.0009" ixz="-0.0007" iyz="0.0"/> -->
-              <inertia
-                  ixx="0.0017" iyy="0.0223" izz="0.0216"
-                  ixy="-0.0009" ixz="-0.0009" iyz="0.0001"/>
+                  ixx="0.001491" iyy="0.019199" izz="0.018359"
+                  ixy="-0.000820" ixz="-0.000019" iyz="0.000079"/>
             </inertial>
             <xacro:link_model type="baselink" />
@@ -56,13 +44,9 @@
           <xacro:unless value="${baselink}">
             <inertial>
-              <origin xyz="${link_length* 0.5 - 11.42 * 0.001} ${-6.06 * 0.001} ${-14.09 * 0.001}" rpy="0 0 0"/>
-              <mass value="0.8890" />
-              <!-- bad problem: https://github.com/tongtybj/aerial_robot/issues/155
+              <origin xyz="${link_length* 0.5 -0.012690} -0.006060 -0.014760" rpy="0 0 0"/>
+              <mass value="0.889000"/>
               <inertia
-                  ixx="0.0017" iyy="0.02" izz="0.019"
-                  ixy="-0.0009" ixz="-0.0004" iyz="0.0"/> -->
-              <inertia
-                  ixx="0.0013" iyy="0.0194" izz="0.0188"
-                  ixy="-0.0008" ixz="0.0007" iyz="0.0"/>
+                  ixx="0.001488" iyy="0.019499" izz="0.018661"
+                  ixy="-0.000832" ixz="-0.000138" iyz="0.000080"/>
             </inertial>
             <xacro:link_model type="general_link" />
@@ -251,23 +235,4 @@
       </joint>
     </xacro:if>
-    <!-- set the fcu frame -->
-    <xacro:if value="${baselink}">
-      <link name="fc">
-        <inertial>
-          <origin xyz="0 0 0" rpy="0 0 0"/>
-          <mass value="0.00001"/>
-          <inertia
-              ixx="0.000001" ixy="0.0" ixz="0.0"
-              iyy="0.000001" iyz="0.0"
-              izz="0.000002"/>
-        </inertial>
-      </link>
-      <joint name="fc_joint" type="fixed">
-        <child link="fc"/>
-        <parent link="link${self}"/>
-        <origin rpy="0 0 0" xyz="0.316 -0.004 0.043"/>
-        <axis xyz="0 0 1"/>
-      </joint>
-    </xacro:if>
     <!-- hardware interface -->
     <xacro:unless value="${self == child}">
