Commit message: Fix the wrong orientation of realsense in dragon model

File: robots/dragon/robots/quad/upboard_sensors_201911/robot.urdf.xacro (robot description, xacro)
@@ -55,5 +55,5 @@
   </xacro:extra_module>
   <xacro:extra_module name = "realsense1_pose_frame" parent = "realsense_t265_unit" visible = "0" >
-    <origin xyz="0 ${6.5 * 0.001} 0 " rpy="0 0 ${-pi/2}"/>
+    <origin xyz="0 ${6.5 * 0.001} 0 " rpy="${pi} 0 ${-pi/2}"/>
     <inertial>
       <mass value = "0.0" />

Commit message: [Temp] remove realsense t265 from updboard_ensors_201911 model

File: robots/dragon/robots/quad/upboard_sensors_201911/robot.urdf.xacro (robot description, xacro)
@@ -42,5 +42,16 @@
     </xacro:extra_module>
   <!-- end: processor: gps -->
+  <xacro:extra_module name = "sensors_mount" parent = "link2" visible = "0" >
+    <origin rpy="0 0 0" xyz="0.387 -0.069 0"/>
+    <inertial>
+      <origin xyz="0 0 0" rpy="0 0 0"/>
+      <mass value="0.007"/>
+      <inertia
+          ixx="0" iyy="0" izz="0"
+          ixy="0" ixz="0" iyz="0"/>
+    </inertial>
+  </xacro:extra_module>
   <!-- 2.3 side view realsense -->
+  <!--
   <xacro:extra_module name = "realsense_t265_unit" parent = "link2" visible = "1"
                       model_url = "package://dragon/urdf/mesh/sensor/horizontal_realsense_t265_unit.dae" >
@@ -64,5 +75,6 @@
           izz="0.0"/>
     </inertial>
-  </xacro:extra_module>
+    </xacro:extra_module>
+  -->
   <!-- end: processor: side-view realsense -->
 </robot>
