Commit message: add plate-like gripper

File: robots/hydrus_xi/robots/quad/upboard202007.urdf.xacro (robot description, xacro)
@@ -16,3 +16,44 @@
     </inertial>
   </xacro:extra_module>
+  #### gripper ####
+  <xacro:extra_module_collision name = "gripper_plane" parent = "link4" visible = "1"
+                      model_url = "package://hydrus_xi/urdf/mesh/mechanical/door_opening_plate.STL">
+    <origin xyz="0.65 0.06 -0.05" rpy="1.5708 0 -1.5708"/>
+    <inertial>
+      <mass value = "0.100" />
+      <origin xyz="0.06 0.05 0.0035" rpy="0 0 0"/>
+      <inertia
+          ixx="0.0003" ixy="0.0003" ixz="0.0"
+          iyy="0.0005" iyz="0.0"
+          izz="0.0008"/>
+    </inertial>
+    <collision>
+      <geometry>
+        <mesh filename="package://hydrus_xi/urdf/mesh/mechanical/door_opening_plate.STL"/>
+      </geometry>
+    </collision>
+  </xacro:extra_module_collision>
+  <gazebo reference="gripper_plane">
+    <self_collide>true</self_collide>
+  </gazebo>
+  <xacro:extra_module_collision name = "gripper_rod" parent = "link1" visible = "1"
+                      model_url = "package://hydrus_xi/urdf/mesh/mechanical/door_opening_rod_asm.STL">
+    <origin xyz="-0.01 -0.016 -0.012" rpy="0 0 3.1415"/>
+    <inertial>
+      <mass value = "0.04" />
+      <origin xyz="0.066 -0.016 0.01" rpy="0 0 0"/>
+      <inertia
+          ixx="0.0001" ixy="0.0" ixz="0.0"
+          iyy="0.0003" iyz="0.0"
+          izz="0.0003"/>
+    </inertial>
+    <collision>
+      <geometry>
+        <mesh filename="package://hydrus_xi/urdf/mesh/mechanical/door_opening_rod_asm.STL"/>
+      </geometry>
+    </collision>
+  </xacro:extra_module_collision>
+  <gazebo reference="gripper_rod">
+    <self_collide>true</self_collide>
+  </gazebo>
 </robot>

Commit message: update gripper model

File: robots/hydrus_xi/robots/quad/upboard202007.urdf.xacro (robot description, xacro)
@@ -18,6 +18,6 @@
   #### gripper ####
   <xacro:extra_module_collision name = "gripper_plane" parent = "link4" visible = "1"
-                      model_url = "package://hydrus_xi/urdf/mesh/mechanical/door_opening_plate.STL">
-    <origin xyz="0.65 0.06 -0.05" rpy="1.5708 0 -1.5708"/>
+                      model_url = "package://hydrus_xi/urdf/mesh/mechanical/door_opening_unit_plate.STL">
+    <origin xyz="0.582 0.016 0.012" rpy="-1.5708 0 -1.5708"/>
     <inertial>
       <mass value = "0.100" />
@@ -30,5 +30,5 @@
     <collision>
       <geometry>
-        <mesh filename="package://hydrus_xi/urdf/mesh/mechanical/door_opening_plate.STL"/>
+        <mesh filename="package://hydrus_xi/urdf/mesh/mechanical/door_opening_unit_plate.STL"/>
       </geometry>
     </collision>
@@ -38,6 +38,6 @@
   </gazebo>
   <xacro:extra_module_collision name = "gripper_rod" parent = "link1" visible = "1"
-                      model_url = "package://hydrus_xi/urdf/mesh/mechanical/door_opening_rod_asm.STL">
-    <origin xyz="-0.01 -0.016 -0.012" rpy="0 0 3.1415"/>
+                      model_url = "package://hydrus_xi/urdf/mesh/mechanical/door_opening_T_long_diff.STL">
+    <origin xyz="-0.007 -0.016 0.012" rpy="-1.5708 0 1.5708"/>
     <inertial>
       <mass value = "0.04" />
@@ -50,5 +50,5 @@
     <collision>
       <geometry>
-        <mesh filename="package://hydrus_xi/urdf/mesh/mechanical/door_opening_rod_asm.STL"/>
+        <mesh filename="package://hydrus_xi/urdf/mesh/mechanical/door_opening_T_long_diff.STL"/>
       </geometry>
     </collision>

Commit message: fix model so that it fits with real machine

File: robots/hydrus_xi/robots/quad/upboard202007.urdf.xacro (robot description, xacro)
@@ -17,7 +17,7 @@
   </xacro:extra_module>
   #### gripper ####
-  <xacro:extra_module_collision name = "gripper_plane" parent = "link4" visible = "1"
+  <xacro:extra_module_collision name = "gripper_plane" parent = "link1" visible = "1"
                       model_url = "package://hydrus_xi/urdf/mesh/mechanical/door_opening_unit_plate.STL">
-    <origin xyz="0.582 0.016 0.012" rpy="-1.5708 0 -1.5708"/>
+    <origin xyz="-0.017 -0.016 0.012" rpy="-1.5708 0 1.5708"/>
     <inertial>
       <mass value = "0.100" />
@@ -37,7 +37,7 @@
     <self_collide>true</self_collide>
   </gazebo>
-  <xacro:extra_module_collision name = "gripper_rod" parent = "link1" visible = "1"
+  <xacro:extra_module_collision name = "gripper_rod" parent = "link4" visible = "1"
                       model_url = "package://hydrus_xi/urdf/mesh/mechanical/door_opening_T_long_diff.STL">
-    <origin xyz="-0.007 -0.016 0.012" rpy="-1.5708 0 1.5708"/>
+    <origin xyz="0.582 0.016 0.012" rpy="-1.5708 0 -1.5708"/>
     <inertial>
       <mass value = "0.04" />

Commit message: gain friction and some

File: robots/hydrus_xi/robots/quad/upboard202007.urdf.xacro (robot description, xacro)
@@ -57,3 +57,8 @@
     <self_collide>true</self_collide>
   </gazebo>
+  <gazebo reference="gripper_plane">
+    <material>Gazebo/Black</material>
+    <mu1 value="5" />
+    <mu2 value="5" />
+  </gazebo>
 </robot>

Commit message: fix model weight and add rosbag play launch

File: robots/hydrus_xi/robots/quad/upboard202007.urdf.xacro (robot description, xacro)
@@ -41,5 +41,5 @@
     <origin xyz="0.582 0.016 0.012" rpy="-1.5708 0 -1.5708"/>
     <inertial>
-      <mass value = "0.04" />
+      <mass value = "0.100" />
       <origin xyz="0.066 -0.016 0.01" rpy="0 0 0"/>
       <inertia

File: robots/hydrus_xi/urdf/link.urdf.xacro (robot description, xacro)
@@ -51,5 +51,5 @@
       <inertial>
         <origin xyz="-0.006114 0.000001 0.032778" rpy="0 0 0"/>
-        <mass value="0.140963"/>
+        <mass value="0.260"/>
         <inertia
             ixx="0.001" iyy="0.001" izz="0.001"

Commit message: fix weight of the gripper

File: robots/hydrus_xi/robots/quad/upboard202007.urdf.xacro (robot description, xacro)
@@ -21,5 +21,5 @@
     <origin xyz="-0.017 -0.016 0.012" rpy="-1.5708 0 1.5708"/>
     <inertial>
-      <mass value = "0.100" />
+      <mass value = "0.070" />
       <origin xyz="0.06 0.05 0.0035" rpy="0 0 0"/>
       <inertia
@@ -41,5 +41,5 @@
     <origin xyz="0.582 0.016 0.012" rpy="-1.5708 0 -1.5708"/>
     <inertial>
-      <mass value = "0.100" />
+      <mass value = "0.075" />
       <origin xyz="0.066 -0.016 0.01" rpy="0 0 0"/>
       <inertia

Commit message: change gazebo model into hinged version and delete camera link

File: robots/hydrus_xi/robots/quad/upboard202007.urdf.xacro (robot description, xacro)
@@ -17,5 +17,5 @@
   </xacro:extra_module>
   #### gripper ####
-  <xacro:extra_module_collision name = "gripper_plane" parent = "link1" visible = "1"
+  <!--xacro:extra_module_collision name = "gripper_plane" parent = "link1" visible = "1"
                       model_url = "package://hydrus_xi/urdf/mesh/mechanical/door_opening_unit_plate.STL">
     <origin xyz="-0.017 -0.016 0.012" rpy="-1.5708 0 1.5708"/>
@@ -36,5 +36,5 @@
   <gazebo reference="gripper_plane">
     <self_collide>true</self_collide>
-  </gazebo>
+  </gazebo-->
   <xacro:extra_module_collision name = "gripper_rod" parent = "link4" visible = "1"
                       model_url = "package://hydrus_xi/urdf/mesh/mechanical/door_opening_T_long_diff.STL">

File: robots/hydrus_xi/urdf/link.urdf.xacro (robot description, xacro)
@@ -112,4 +112,39 @@
         <axis xyz="0 0 1"/>
       </joint>
+    </xacro:if>
+    ## environmental adherence plate passive joint
+    <xacro:if value="${self == 1}">
+      <link name="wall_hinge">
+        <origin xyz="0 0 0" rpy="0 0 0"/>
+        <inertial>
+          <mass value = "0.070" />
+          <origin xyz="0 0 0" rpy="0 0 0"/>
+          <inertia
+              ixx="0.0003" ixy="0.0003" ixz="0.0"
+              iyy="0.0005" iyz="0.0"
+              izz="0.0008"/>
+        </inertial>
+        <collision>
+          <geometry>
+            <mesh filename="package://hydrus_xi/urdf/mesh/mechanical/door_opening_plate_hinge.STL"/>
+          </geometry>
+        </collision>
+        <visual>
+          <geometry>
+            <mesh filename="package://hydrus_xi/urdf/mesh/mechanical/door_opening_plate_hinge.STL"/>
+          </geometry>
+        </visual>
+      </link>
+      <joint name="hinge_joint" type="revolute">
+        <parent link="link1"/>
+        <child link="wall_hinge"/>
+        <origin xyz="-0.04 0 0" rpy="0 0 3.1415"/>
+        <limit lower="-1.5" upper="1.5" effort="100" velocity="100"/>
+        <axis xyz="0 0 1"/>
+        <dynamics damping="0.01" friction="0.01"/>
+      </joint>
+      <gazebo reference="wall_hinge">
+        <self_collide>true</self_collide>
+      </gazebo>
     </xacro:if>
     #### joints ####
