Commit message: modify collision

File: robots/hydrus_xi/urdf/link.urdf.xacro (robot description, xacro)
@@ -59,10 +59,14 @@
         <origin xyz="0 0 0" rpy="0 0 0"/>
       </xacro:mesh_model>
-      <!-- <collision> -->
-      <!--   <origin rpy="0 0 0" xyz="0 0 ${- collision_rotor_height / 2}"/> -->
-      <!--   <geometry> -->
-      <!--     <cylinder length="${collision_rotor_height}" radius="${protector_radius + 0.01}"/> -->
-      <!--   </geometry> -->
-      <!-- </collision> -->
+      <collision>
+        <origin rpy="0 0 0" xyz="0 0 0"/>
+        <geometry>
+          <mesh filename="package://hydrus_xi/urdf/mesh/link/propeller_link.dae"/>
+        </geometry>
+        <!--origin rpy="0.3 0 0" xyz="0 0 ${- collision_rotor_height / 2}"/-->
+        <!--geometry-->
+          <!--cylinder length="${collision_rotor_height}" radius="${protector_radius + 0.01}"/-->
+        <!--/geometry-->
+      </collision>
     </link>
     <xacro:damping_factor link="gimbal_link${self}"/>

Commit message: changed joit config

File: robots/hydrus_xi/urdf/link.urdf.xacro (robot description, xacro)
@@ -117,5 +117,5 @@
     <xacro:unless value="${self == child}">
       <joint name="joint${self}" type="revolute">
-        <limit effort="3.3" lower="-1.57" upper="1.57" velocity="0.5"/>
+        <limit effort="5" lower="-1.57" upper="1.57" velocity="0.5"/>
         <parent link="link${self}"/>
         <child link="link${child}"/>

Commit message: ball joint

File: robots/hydrus_xi/urdf/link.urdf.xacro (robot description, xacro)
@@ -115,11 +115,23 @@
     ## environmental adherence plate passive joint
     <xacro:if value="${self == 1}">
+      <link name="virt_ball1">
+        <inertial>
+          <mass value="0.030"/>
+          <inertia ixx="5.8083e-4" ixy="0" ixz="0" iyy="3.0833e-5" iyz="0" izz="5.9083e-4" />
+        </inertial>
+      </link>
+      <link name="virt_ball2">
+        <inertial>
+          <mass value="0.030"/>
+          <inertia ixx="5.8083e-4" ixy="0" ixz="0" iyy="3.0833e-5" iyz="0" izz="5.9083e-4" />
+        </inertial>
+      </link>
       <link name="wall_hinge">
         <origin xyz="0 0 0" rpy="0 0 0"/>
         <inertial>
-          <mass value = "0.070" />
-          <origin xyz="0 0 0" rpy="0 0 0"/>
-          <inertia
-              ixx="0.0003" ixy="0.0003" ixz="0.0"
+          <mass value = "0.030" />
+          <origin xyz="0 0 0" rpy="0 0 0"/>
+          <inertia
+              ixx="0.0005" ixy="0.0" ixz="0.0"
               iyy="0.0005" iyz="0.0"
               izz="0.0008"/>
@@ -136,8 +148,22 @@
         </visual>
       </link>
+      <joint name="virt_roll_joint" type="revolute">
+        <parent link="link1"/>
+        <child link="virt_ball1"/>
+        <origin xyz="-0.04 0 0" rpy="0 0 3.1415"/>
+        <limit lower="-0.3" upper="0.3" effort="100" velocity="100"/>
+        <axis xyz="1 0 0"/>
+        <dynamics damping="0.01" friction="0.01"/>
+      </joint>
+      <joint name="virt_pitch_joint" type="revolute">
+        <parent link="virt_ball1"/>
+        <child link="virt_ball2"/>
+        <limit lower="-0.3" upper="0.3" effort="100" velocity="100"/>
+        <axis xyz="0 1 0"/>
+        <dynamics damping="0.01" friction="0.01"/>
+      </joint>
       <joint name="hinge_joint" type="revolute">
-        <parent link="link1"/>
+        <parent link="virt_ball2"/>
         <child link="wall_hinge"/>
-        <origin xyz="-0.04 0 0" rpy="0 0 3.1415"/>
         <limit lower="-1.5" upper="1.5" effort="100" velocity="100"/>
         <axis xyz="0 0 1"/>
