Commit message: [Twin Hammer][urdf] Create new arg to switch using dummy weight

File: robots/twin_hammer/urdf/device_with_dummy_weight.urdf.xacro (robot description, xacro)
@@ -260,5 +260,5 @@
  </joint>
  <!-- when fix main body  -->
- <!-- <link name="dummy_weight">
+ <link name="dummy_weight">
     <inertial>
       <origin xyz="0 0 0" rpy="0 0 0"/>
@@ -280,5 +280,5 @@
     <child link="root"/>
     <origin rpy="0 0 0" xyz="0 0 1.0"/>
-  </joint> -->
+  </joint>
   <!-- ft_sensor_gazebo joint -->
   <!-- <joint name="root_to_dummyweight_joint" type="fixed">
