Commit message: [Twin Hammer] [urdf] [controller] Change the direction of frame of gimbal unit 2

File: robots/twin_hammer/urdf/device.urdf.xacro (robot description, xacro)
@@ -55,5 +55,5 @@
      </xacro:if>
      <xacro:if value="${id == 2}" >
-       <origin rpy="0 0 0" xyz="${gimbal_roll_x_offset - rod_length*0.5} 0 0"/>
+       <origin rpy="0 0 ${pi}" xyz="${gimbal_roll_x_offset - rod_length*0.5} 0 0"/>
      </xacro:if>
      <axis xyz="1 0 0"/>

File: robots/twin_hammer/urdf/device_with_dummy_weight.urdf.xacro (robot description, xacro)
@@ -55,5 +55,5 @@
      </xacro:if>
      <xacro:if value="${id == 2}" >
-       <origin rpy="0 0 0" xyz="${gimbal_roll_x_offset - rod_length*0.5} 0 0"/>
+       <origin rpy="0 0 ${pi}" xyz="${gimbal_roll_x_offset - rod_length*0.5} 0 0"/>
      </xacro:if>
      <axis xyz="1 0 0"/>
