Commit message: [Beetle_Hand] [urdf] Change mass and inertia

File: robots/beetle/urdf/beetle_hand.urdf.xacro (robot description, xacro)
@@ -24,9 +24,9 @@
       <inertial>
         <origin xyz="0.000169 0.002346 0.106123" rpy="0 0 0"/>
-        <mass value="1.400000"/>
-        <inertia
-            ixx="0.024393" ixy="0.00005" ixz="0.000015"
-	    iyy="0.024541" iyz="0.000205"
-	    izz="0.043817"/>
+        <mass value="1.37825"/>
+        <inertia
+            ixx="0.046756" ixy="0.000586" ixz="0.000055"
+	    iyy="0.063216" iyz="0.000219"
+	    izz="0.058783"/>
       </inertial>
       <visual>
